File: sbc09_debugger.kicad_sch (KiCad schematic)
At the start: 7 parts, among them J1 Conn_02x10_Odd_Even, J2 Conn_02x10_Odd_Even, J3 Conn_02x25_Odd_Even

Commit message: Use backplane pin numbering and the correct male IDC footprint
Parts:
- C1: footprint (none) -> Capacitor_THT:C_Disc_D4.7mm_W2.5mm_P5.00mm
Connections:
- net A0: now also J3.33 (Pin_33); no longer J3.18 (Pin_18)
- net A1: now also J3.34 (Pin_34); no longer J3.17 (Pin_17)
- net A2: now also J3.35 (Pin_35); no longer J3.16 (Pin_16)
- net A3: now also J3.36 (Pin_36); no longer J3.15 (Pin_15)
- net BA: now also J3.13 (Pin_13); no longer J3.38 (Pin_38)
- net BS: now also J3.21 (Pin_21); no longer J3.30 (Pin_30)
- net D0: now also J3.25 (Pin_25); no longer J3.26 (Pin_26)
- net D1: now also J3.26 (Pin_26); no longer J3.25 (Pin_25)
- net D2: now also J3.27 (Pin_27); no longer J3.24 (Pin_24)
- net D3: now also J3.28 (Pin_28); no longer J3.23 (Pin_23)
- net D4: now also J3.29 (Pin_29); no longer J3.22 (Pin_22)
- net D5: now also J3.30 (Pin_30); no longer J3.21 (Pin_21)
- net D6: now also J3.31 (Pin_31); no longer J3.20 (Pin_20)
- net D7: now also J3.32 (Pin_32); no longer J3.19 (Pin_19)
- net GND: now also J3.3 (Pin_3), J3.4 (Pin_4), J3.50 (Pin_50); no longer J3.1 (Pin_1), J3.47 (Pin_47), J3.48 (Pin_48)
- net LIC: now also J3.6 (Pin_6); no longer J3.45 (Pin_45)
- net RnW: now also J3.18 (Pin_18); no longer J3.33 (Pin_33)
- net at R1.1: now also J3.1 (Pin_1); no longer J3.50 (Pin_50)
Other:
- moved on the sheet: J3
Changed lines of the file:
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@@
       (effects (font (size 1.27 1.27)) (justify left))
     )
-    (property "Footprint" "" (id 2) (at 96.52 119.38 0)
+    (property "Footprint" "Capacitor_THT:C_Disc_D4.7mm_W2.5mm_P5.00mm" (id 2) (at 96.52 119.38 0)
       (effects (font (size 1.27 1.27)) hide)
     )
@@
     (pin "2")
   )
-  (symbol (lib_id "Connector_Generic:Conn_02x25_Odd_Even") (at 64.77 83.82 0) (unit 1)
+  (symbol (lib_id "Connector_Generic:Conn_02x25_Odd_Even") (at 67.31 83.82 180) (unit 1)
     (in_bom yes) (on_board yes) (fields_autoplaced)
     (property "Reference" "J3" (id 0) (at 66.04 46.99 0))
     (property "Value" "Conn_02x25_Odd_Even" (id 1) (at 66.04 49.53 0))
-    (property "Footprint" "" (id 2) (at 64.77 83.82 0)
-      (effects (font (size 1.27 1.27)) hide)
-    )
-    (property "Datasheet" "~" (id 3) (at 64.77 83.82 0)
+    (property "Footprint" "" (id 2) (at 67.31 83.82 0)
+      (effects (font (size 1.27 1.27)) hide)
+    )
+    (property "Datasheet" "~" (id 3) (at 67.31 83.82 0)
       (effects (font (size 1.27 1.27)) hide)
     )
@@
     )
     (path "/d3bd2f73-786f-472c-89b7-10fd054df22c"
-      (reference "J3") (unit 1) (value "Conn_02x25_Odd_Even") (footprint "Connector_PinSocket_2.54mm:PinSocket_2x25_P2.54mm_Horizontal")
+      (reference "J3") (unit 1) (value "Conn_02x25_Odd_Even") (footprint "Connector_IDC:IDC-Header_2x25_P2.54mm_Horizontal")
     )
     (path "/fbcf0fbf-a72b-440f-a386-5cbf59a50354"
